File: hardware/sheets/rails.kicad_sch (KiCad schematic)
At the start: 0 parts

Commit message: hw(rails): finish the rails sheet and fix four defects found on review
The drafting agent's topology was sound but it stopped before finishing, and
verification against the primary datasheets turned up four real problems.

Constant-on-time loop had no ripple to work with.  The LM5164 needs >= 20 mV of
ripple AT FB (datasheet 6.2); an all-ceramic output stage with a feedforward cap
delivered ~3 mV, a 6.5x shortfall.  Replaced with the datasheet's Type-3
injection network on both rails, sized from equations 24-26 and checked against
the >= 12 mV at minimum VIN criterion.  Chosen over adding series ESR because
the ADC sense chain runs off these rails.

Both enables were missing their mandatory pulldowns.  EN_3V3SW and EN_BOOST
reached their pins with nothing else on the net, against the plan's
passive-default table and the LM51571's own "must not be left floating".
Added R19/R20.

The switched 3.3 V rail did not exist.  The load-switch block was dropped when
the sheet was restructured around the boost; added as block 4 with the
DML3017LDC, its mandatory external BLEED resistor and CSR cap.

Symbol pin types were generating false ERC violations -- SW was typed power_in,
so ERC demanded an external driver for the converter's own switch node.

Also corrects two claims in part-selection.md that were written from the feature
list rather than the pin table: the BLEED resistor is external and mandatory,
not an on-chip 100 ohm, and PG is tied to GND rather than pulled up, because a
100k pullup would burn 33 uA of a 100 uA sleep budget.

ERC 26 violations -> 6, all six being root sheet pins whose counterparts live on
mcu_can and outputs, which are not drawn yet.  Netlist verified independently:
VBAT and VLOGIC_IN now span both sheets, EN_3V3SW gates both switched rails, and
the Type-3 nodes are correct on both bucks.

Co-Authored-By: Claude Opus 5 <noreply@anthropic.com>
Claude-Session: https://claude.ai/code/session_01Bkq7QP4he4cdfxkUNzx7DL
Parts:
- added C10, C11, C16: 22uF, symbol Device:C
- added C12, C6: 2.2uF, symbol Device:C
- added C13, C17, C27, C33, C7: 100nF, symbol Device:C
- added C14, C28, C29, C8: 2.2nF, symbol Device:C
- added C15: 39pF, symbol Device:C
- added C18, C19, C34: 10uF, symbol Device:C
- added C20, C21, C22: 4.7uF, symbol Device:C
- added C23: 10nF, symbol Device:C
- added C24: 100pF, symbol Device:C
- added C25: 22nF, symbol Device:C
- added C26, C30, C31: 1uF, symbol Device:C
- added C32: 1nF, symbol Device:C
- added C9: 68pF, symbol Device:C
- added D4: SS5PH102, symbol Device:D_Schottky
- added L3: 6.8uH XAL4030-682ME, symbol Device:L
- added L4, L5: 22uH, symbol Device:L
- added R10: 9.09k, symbol Device:R
- added R11: 37.4k, symbol Device:R
- added R12: 115k, symbol Device:R
- added R13: 4.99k, symbol Device:R
- added R14: 2.61k, symbol Device:R
- added R15: 5.1R, symbol Device:R
- added R16: 0R, symbol Device:R
- added R17: 133k, symbol Device:R
- added R18: 174k, symbol Device:R
- added R19, R20: 100k, symbol Device:R
- added R21: 100R, symbol Device:R
- added R4: 20.5k, symbol Device:R
- added R5: 348k, symbol Device:R
- added R6, R9: 200k, symbol Device:R
- added R7: 31.6k, symbol Device:R
- added R8: 634k, symbol Device:R
- added U1, U2: LM5164DDA, symbol Regulator_Switching:LM5164DDA
- added U3: LM51571-Q1, symbol mccan_parts:LM51571QRTERQ1
- added U4: DML3017LDC, symbol mccan_parts:DML3017LDC
Connections:
- new net: C15.2, C29.1, R18.2
- new net: R15.1, U3.2 (VCC)
- new net: C26.1, R15.2
- new net: R11.1, U3.11 (MODE)
- new net: C14.1, U2.7 (BST)
- new net: C25.1, U3.10 (SS)
- new net: C24.1, R14.1, U3.8 (COMP)
- new net: C23.1, R14.2
- new net: R10.1, U3.5 (RT)
- new net: C28.1, C9.2, R17.2
- new net: R4.1, U1.4 (RON)
- new net: R21.2, U4.7 (BLEED)
- new net: R7.1, U2.4 (RON)
- new net: C8.1, U1.7 (BST)
- new net: C32.1, U4.5 (SR)
- new net: C27.1, R16.2, U3.3 (BIAS)
- new net +24V: C20.1, C21.1, C22.1, D4.1 (K), R12.1
- new net +3V3_ALW: C10.1, C11.1, C28.2, C30.1, C31.1, L4.2, R5.1, U4.1 (VIN), U4.13 (VIN), U4.3 (VCC)
- new net +3V3_SW: C33.1, C34.1, R21.1, U4.10 (VOUT), U4.11 (VOUT), U4.12 (VOUT), U4.8 (VOUT), U4.9 (VOUT)
- new net +5V: C16.1, C17.1, C29.2, L5.2, R8.1
- new net EN_3V3SW: R19.1, U2.3 (EN/UVLO), U4.2 (EN)
- new net EN_BOOST: R20.1, U3.6 (EN_UVLO_SYNC)
- new net FB_24V: R12.2, R13.1, U3.9 (FB)
- new net FB_3V3: C9.1, R5.2, R6.1, U1.5 (FB)
- new net FB_5V: C15.1, R8.2, R9.1, U2.5 (FB)
- new net GND: C10.2, C11.2, C12.2, C13.2, C16.2, C17.2, C18.2, C19.2, C20.2, C21.2, C22.2, C23.2, C24.2, C25.2, C26.2, C27.2, C30.2, C31.2, C32.2, C33.2, C34.2, C6.2, C7.2, R10.2, R11.2, R13.2, R19.2, R20.2, R4.2, R6.2, R7.2, R9.2, U1.1 (GND), U1.9 (EP), U2.1 (GND), U2.9 (EP), U3.1 (PGND), U3.16 (PGND), U3.17 (EP), U3.7 (AGND), U4.4 (GND), U4.6 (PG)
- new net SW_3V3: C8.2, L4.1, R17.1, U1.8 (SW)
- new net SW_5V: C14.2, L5.1, R18.1, U2.8 (SW)
- new net SW_BOOST: D4.2 (A), L3.2, U3.12 (SW), U3.13 (SW), U3.14 (SW)
- new net VBAT: C12.1, C13.1, C18.1, C19.1, L3.1, R16.1, U2.2 (VIN)
- new net VLOGIC_IN: C6.1, C7.1, U1.2 (VIN), U1.3 (EN/UVLO)
- no-connect marks 0 -> 4
