File: hardware/sheets/mcu_can.kicad_sch (KiCad schematic)
At the start: 0 parts

Commit message: hw(sch): ESP32-WROOM-32E-N8, TJA1042 listen-only, prog header (Task 5)
The mcu_can sheet, with every net verified from the exported netlist rather than
from the drawing.  All 24 GPIO assignments match the plan's Global Constraints
table pin for pin.

Listen-only is structural, not a setting.  The netlist shows GPIO 17 reaching
only R23, and the transceiver TXD reaching only R23 and its pull-up, so the DNP
0 ohm link is the single conductive path and a board built to the BOM cannot
assert a dominant bit on the vehicle bus.

The transceiver's two supplies are deliberately split: VIO on +3V3_ALW keeps the
receiver alive so bus traffic still pulls RXD low for EXT0 wake, while VCC on the
switched +5V powers down the transmit side in sleep.  Both pull-ups (TXD, STB)
rest high, so neither costs anything against the sleep budget.

The root schematic is now generated rather than patched, from a declaration of
boxes and pins, with the four sheet UUIDs pinned -- changing one would orphan
every reference designator on that sheet.  Sheet pins join through root-level
labels on stubs; with ~40 inter-sheet nets, wires drawn between the boxes are an
unreadable rat's nest.

Two mechanical defect classes found and now asserted against in the generators:
coordinates must be exact multiples of 1.27 mm (a pin that misses its wire by
0.6 mm looks connected and is not -- 161 instances), and a local label must sit
at a wire's end rather than mid-wire, which forms the net but leaves the endpoint
dangling (14 instances).

Three additions beyond the plan, all flagged in part-selection.md rather than
smuggled in: a pulldown on GPIO 12 (it selects flash voltage at boot and the plan
would have left the strap floating), the new net name IGN_IN for the
ignition-switched sense wire, and putting the MUX/DSEL/DIAG pulldowns on this
sheet because MUX_S3 is GPIO 5, a strapping pin sampled at reset.

ERC: 25 violations, every one of them the outputs sheet not existing yet.

Co-Authored-By: Claude Opus 5 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
Parts:
- added C35: 10uF, symbol Device:C
- added C36, C38, C39: 100nF, symbol Device:C
- added C37: 1uF, symbol Device:C
- added D5: green, symbol Device:LED
- added D6, D7: 24V bidir, symbol Device:D_TVS
- added D8: BAT54, symbol Device:D_Schottky
- added J2: Prog/UART, symbol Connector_Generic:Conn_01x06
- added L6: 51uH CM choke, symbol Device:L_Coupled
- added Q2, Q3: MMBT3904, symbol Transistor_BJT:Q_NPN_BEC
- added R22, R24, R25, R28, R29, R30, R31, R32, R33, R34, R35, R36: 10k, symbol Device:R
- added R23: 0R, symbol Device:R
- added R26: 120R, symbol Device:R
- added R27: 1k, symbol Device:R
- added R37: 90.9k, symbol Device:R
- added R38: 33k, symbol Device:R
- added R39: 100k, symbol Device:R
- added SW1: BOOT, symbol Switch:SW_Push
- added SW2: EN/RESET, symbol Switch:SW_Push
- added U5: ESP32-WROOM-32E-N8, symbol RF_Module:ESP32-WROOM-32E
- added U6: TJA1042T/3, symbol Interface_CAN_LIN:TJA1042T-3
Connections:
- new net: R23.2, R24.2, U6.1 (TXD)
- new net: Q2.1 (B), R28.2
- new net: Q3.1 (B), R29.2
- new net: L6.1, U6.7 (CANH)
- new net: L6.3, U6.6 (CANL)
- new net: D5.2 (A), R27.1
- new net +3V3_ALW: C35.1, C36.1, C39.1, D8.1 (K), J2.1 (Pin_1), R22.1, R24.1, R25.1, U5.2 (VDD), U6.5 (VIO)
- new net +5V: C38.1, U6.3 (VCC)
- new net BOOT_N: Q3.3 (C), SW1.1, U5.25 (IO0)
- new net CANH: D6.1 (A1), L6.2, R26.1
- new net CANL: D7.1 (A1), L6.4, R26.2
- new net CAN_RXD: U5.7 (IO35), U6.4 (RXD)
- new net CAN_STB: R25.2, U5.13 (IO14), U6.8 (STB)
- new net CAN_TXD: R23.1, U5.28 (IO17)
- new net DEN_DSEL: R34.1, U5.9 (IO33)
- new net DTR: J2.5 (Pin_5), Q2.2 (E), R29.1
- new net EN_3V3SW: U5.11 (IO26)
- new net EN_BOOST: U5.10 (IO25)
- new net EN_DIAG: R35.1, U5.12 (IO27)
- new net EN_MCU: C37.1, Q2.3 (C), R22.2, SW2.1, U5.3 (EN)
- new net GND: C35.2, C36.2, C37.2, C38.2, C39.2, D5.1 (K), D6.2 (A2), D7.2 (A2), J2.2 (Pin_2), R30.2, R31.2, R32.2, R33.2, R34.2, R35.2, R36.2, R38.2, R39.2, SW1.2, SW2.2, U5.[1,15,38,39] (GND), U6.2 (GND)
- new net I2C_SCL: U5.36 (IO22)
- new net I2C_SDA: U5.33 (IO21)
- new net IGN_IN: R37.1
- new net IGN_SENSE: D8.2 (A), R37.2, R38.1, R39.1, U5.4 (SENSOR_VP)
- new net IO12_STRAP: R36.1, U5.14 (IO12)
- new net ISNS_DEN: U5.6 (IO34)
- new net LED_STAT: R27.2, U5.16 (IO13)
- new net MUX_S0: R30.1, U5.37 (IO23)
- new net MUX_S1: R31.1, U5.26 (IO4)
- new net MUX_S2: R32.1, U5.27 (IO16)
- new net MUX_S3: R33.1, U5.29 (IO5)
- new net PWM_DEN_A: U5.30 (IO18)
- new net PWM_DEN_B: U5.31 (IO19)
- new net RGB_ISNS: U5.8 (IO32)
- new net RTS: J2.6 (Pin_6), Q3.2 (E), R28.1
- new net UART_RX: J2.4 (Pin_4), U5.34 (RXD0/IO3)
- new net UART_TX: J2.3 (Pin_3), U5.35 (TXD0/IO1)
- no-connect marks 0 -> 3

Commit message: hw: J1 to 3-way, IGN_IN on cavity 1 for the battery-feed topology
The Experia's peripheral outlet closes all 12 V at shut-off, so the shipped build
(topology A) needs no ignition signal at all.  This provisions the third cavity
so a battery-fed installation (topology B) is a harness change plus populating
R37/R38, rather than a new panel: Superseal 1.5 2-way and 3-way are different
cutouts, so it could not have been retrofitted.

The third cavity went ABOVE the existing two, not below.  GND_IN drops vertically
from pin 2 at x=31.75 down to y=101.6, so a pin placed below would have landed on
that wire and shorted IGN_IN to ground.  Placing it above left every existing
wire, junction and net on this verified sheet untouched.  Verified from the
netlist: FEED_P and GND_IN keep exactly their previous membership, and GND_IN is
still separate from GND, so the common-mode choke split is intact.  The pins
renumber as a consequence - 1 = IGN_IN, 2 = +12 V, 3 = GND - and cavity 1 being
an end cavity is the easy one to plug.

Adds C40, 100 nF on IGN_SENSE.  IGN_IN is an unshielded 12 V wire entering a
sealed enclosure onto a high-impedance node; C40 forms an RC with R37 giving
tau ~ 2 ms, which costs nothing against an ignition signal that changes over
seconds.  Flagged in part-selection.md as an addition.

Also records a real inconsistency found on the way: power_input has no working
generator.  The scratchpad gen.py lost its notes module to a filename collision,
and once reconstructed it emitted a materially different file from the committed
sheet, so this change was made by surgical text edit and the stale generator was
deliberately not committed.

ERC 25 -> 23 violations; the two IGN_IN single-pin warnings cleared now that the
net has a real source and a real consumer.  The remaining 23 are all the outputs
sheet, which does not exist yet.

Co-Authored-By: Claude Opus 5 <noreply@anthropic.com>
Claude-Session: https://claude.ai/code/session_01Bkq7QP4he4cdfxkUNzx7DL
Parts:
- added C40: 100nF, symbol Device:C
Connections:
- net GND: now also C40.2
- net IGN_SENSE: now also C40.1
Changed lines of the file:
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@@
 	)
 	(junction
+		(at 78.74 111.76)
+		(diameter 0)
+		(color 0 0 0 0)
+	)
+	(junction
 		(at 109.22 76.2)
 		(diameter 0)
@@
 	(wire
 		(pts
-			(xy 72.39 111.76) (xy 83.82 111.76)
+			(xy 72.39 111.76) (xy 78.74 111.76)
+		)
+		(stroke
+			(width 0)
+			(type default)
+		)
+	)
+	(wire
+		(pts
+			(xy 78.74 111.76) (xy 83.82 111.76)
 		)
 		(stroke
@@
 	)
 	(symbol
+		(lib_id "Device:C")
+		(at 78.74 115.57 0)
+		(unit 1)
+		(body_style 1)
+		(exclude_from_sim no)
+		(in_bom yes)
+		(on_board yes)
+		(in_pos_files yes)
+		(dnp no)
+		(property "Reference" "C40"
+			(at 80.391 114.3 0)
+			(show_name no)
+			(do_not_autoplace no)
+			(effects
+				(font
+					(size 1.27 1.27)
+				)
+				(justify left)
+			)
+		)
+		(property "Value" "100nF"
+			(at 80.391 116.84 0)
+			(show_name no)
+			(do_not_autoplace no)
+			(effects
+				(font
+					(size 1.27 1.27)
+				)
+				(justify left)
+			)
+		)
+		(property "Footprint" ""
+			(at 78.74 115.57 0)
+			(hide yes)
+			(show_name no)
+			(do_not_autoplace no)
+			(effects
+				(font
+					(size 1.27 1.27)
+				)
+			)
+		)
+		(property "Datasheet" ""
+			(at 78.74 115.57 0)
+			(hide yes)
+			(show_name no)
+			(do_not_autoplace no)
+			(effects
+				(font
+					(size 1.27 1.27)
+				)
+			)
+		)
+		(property "Description" ""
+			(at 78.74 115.57 0)
+			(hide yes)
+			(show_name no)
+			(do_not_autoplace no)
+			(effects
+				(font
+					(size 1.27 1.27)
+				)
+			)
+		)
+		(pin "1"
+		)
+		(pin "2"
+		)
+		(instances
+			(project "mccan"
+				(path "/7410bb74-5653-4f1b-8c7c-ce17eb633f20/5a511665-9b85-4ced-b6e3-f23e247294e2"
+					(reference "C40")
+					(unit 1)
+				)
+			)
+		)
+	)
+	(symbol
+		(lib_id "power:GND")
+		(at 78.74 119.38 0)
+		(unit 1)
+		(body_style 1)
+		(exclude_from_sim no)
+		(in_bom yes)
+		(on_board yes)
+		(in_pos_files yes)
+		(dnp no)
+		(property "Reference" "#PWR216"
+			(at 78.74 125.73 0)
+			(hide yes)
+			(show_name no)
+			(do_not_autoplace no)
+			(effects
+				(font
+					(size 1.27 1.27)
+				)
+				(justify left)
+			)
+		)
+		(property "Value" "GND"
+			(at 78.74 123.19 0)
+			(hide yes)
+			(show_name no)
+			(do_not_autoplace no)
+			(effects
+				(font
+					(size 1.27 1.27)
+				)
+				(justify left)
+			)
+		)
+		(property "Footprint" ""
+			(at 78.74 119.38 0)
+			(hide yes)
+			(show_name no)
+			(do_not_autoplace no)
+			(effects
+				(font
+					(size 1.27 1.27)
+				)
+			)
+		)
+		(property "Datasheet" ""
+			(at 78.74 119.38 0)
+			(hide yes)
+			(show_name no)
+			(do_not_autoplace no)
+			(effects
+				(font
+					(size 1.27 1.27)
+				)
+			)
+		)
+		(property "Description" "Power symbol creates a global label with name \"GND\" , ground"
+			(at 78.74 119.38 0)
+			(hide yes)
+			(show_name no)
+			(do_not_autoplace no)
+			(effects
+				(font
+					(size 1.27 1.27)
+				)
+			)
+		)
+		(pin "1"
+		)
+		(instances
+			(project "mccan"
+				(path "/7410bb74-5653-4f1b-8c7c-ce17eb633f20/5a511665-9b85-4ced-b6e3-f23e247294e2"
+					(reference "#PWR216")
+					(unit 1)
+				)
+			)
+		)
+	)
+	(symbol
 		(lib_id "Device:D_Schottky")
 		(at 83.82 107.95 270)
@@
 		(in_pos_files yes)
 		(dnp no)
-		(property "Reference" "#PWR216"
+		(property "Reference" "#PWR217"
 			(at 40.64 234.95 0)
 			(hide yes)
@@
 			(project "mccan"
 				(path "/7410bb74-5653-4f1b-8c7c-ce17eb633f20/5a511665-9b85-4ced-b6e3-f23e247294e2"
-					(reference "#PWR216")
+					(reference "#PWR217")
 					(unit 1)
 				)
@@
 		(in_pos_files yes)
 		(dnp no)
-		(property "Reference" "#PWR217"
+		(property "Reference" "#PWR218"
 			(at 55.88 234.95 0)
 			(hide yes)
@@
 			(project "mccan"
 				(path "/7410bb74-5653-4f1b-8c7c-ce17eb633f20/5a511665-9b85-4ced-b6e3-f23e247294e2"
-					(reference "#PWR217")
+					(reference "#PWR218")
 					(unit 1)
 				)
@@
 		(in_pos_files yes)
 		(dnp no)
-		(property "Reference" "#PWR218"
+		(property "Reference" "#PWR219"
 			(at 71.12 234.95 0)
 			(hide yes)
@@
 			(project "mccan"
 				(path "/7410bb74-5653-4f1b-8c7c-ce17eb633f20/5a511665-9b85-4ced-b6e3-f23e247294e2"
-					(reference "#PWR218")
+					(reference "#PWR219")
 					(unit 1)
 				)
@@
 		(in_pos_files yes)
 		(dnp no)
-		(property "Reference" "#PWR219"
+		(property "Reference" "#PWR220"
 			(at 86.36 234.95 0)
 			(hide yes)
@@
 			(project "mccan"
 				(path "/7410bb74-5653-4f1b-8c7c-ce17eb633f20/5a511665-9b85-4ced-b6e3-f23e247294e2"
-					(reference "#PWR219")
+					(reference "#PWR220")
 					(unit 1)
 				)
@@
 		(in_pos_files yes)
 		(dnp no)
-		(property "Reference" "#PWR220"
+		(property "Reference" "#PWR221"
 			(at 101.6 234.95 0)
 			(hide yes)
@@
 			(project "mccan"
 				(path "/7410bb74-5653-4f1b-8c7c-ce17eb633f20/5a511665-9b85-4ced-b6e3-f23e247294e2"
-					(reference "#PWR220")
+					(reference "#PWR221")
 					(unit 1)
 				)
@@
 		(in_pos_files yes)
 		(dnp no)
-		(property "Reference" "#PWR221"
+		(property "Reference" "#PWR222"
 			(at 116.84 234.95 0)
 			(hide yes)
@@
 			(project "mccan"
 				(path "/7410bb74-5653-4f1b-8c7c-ce17eb633f20/5a511665-9b85-4ced-b6e3-f23e247294e2"
-					(reference "#PWR221")
+					(reference "#PWR222")
 					(unit 1)
 				)
@@
 		(in_pos_files yes)
 		(dnp no)
-		(property "Reference" "#PWR222"
+		(property "Reference" "#PWR223"
 			(at 132.08 234.95 0)
 			(hide yes)
@@
 			(project "mccan"
 				(path "/7410bb74-5653-4f1b-8c7c-ce17eb633f20/5a511665-9b85-4ced-b6e3-f23e247294e2"
-					(reference "#PWR222")
+					(reference "#PWR223")
 					(unit 1)
 				)
