File: hardware/sheets/power_input.kicad_sch (KiCad schematic)
At the start: 16 parts, among them J1 PWR (SS1.5 2-way), Q1 SQJ415EP

Commit message: hw: J1 to 3-way, IGN_IN on cavity 1 for the battery-feed topology
The Experia's peripheral outlet closes all 12 V at shut-off, so the shipped build
(topology A) needs no ignition signal at all.  This provisions the third cavity
so a battery-fed installation (topology B) is a harness change plus populating
R37/R38, rather than a new panel: Superseal 1.5 2-way and 3-way are different
cutouts, so it could not have been retrofitted.

The third cavity went ABOVE the existing two, not below.  GND_IN drops vertically
from pin 2 at x=31.75 down to y=101.6, so a pin placed below would have landed on
that wire and shorted IGN_IN to ground.  Placing it above left every existing
wire, junction and net on this verified sheet untouched.  Verified from the
netlist: FEED_P and GND_IN keep exactly their previous membership, and GND_IN is
still separate from GND, so the common-mode choke split is intact.  The pins
renumber as a consequence - 1 = IGN_IN, 2 = +12 V, 3 = GND - and cavity 1 being
an end cavity is the easy one to plug.

Adds C40, 100 nF on IGN_SENSE.  IGN_IN is an unshielded 12 V wire entering a
sealed enclosure onto a high-impedance node; C40 forms an RC with R37 giving
tau ~ 2 ms, which costs nothing against an ignition signal that changes over
seconds.  Flagged in part-selection.md as an addition.

Also records a real inconsistency found on the way: power_input has no working
generator.  The scratchpad gen.py lost its notes module to a filename collision,
and once reconstructed it emitted a materially different file from the committed
sheet, so this change was made by surgical text edit and the stale generator was
deliberately not committed.

ERC 25 -> 23 violations; the two IGN_IN single-pin warnings cleared now that the
net has a real source and a real consumer.  The remaining 23 are all the outputs
sheet, which does not exist yet.

Co-Authored-By: Claude Opus 5 <noreply@anthropic.com>
Claude-Session: https://claude.ai/code/session_01Bkq7QP4he4cdfxkUNzx7DL
Parts:
- J1: value PWR (SS1.5 2-way) -> PWR (SS1.5 3-way); symbol Connector:Conn_01x02_Pin -> Connector:Conn_01x03_Pin
Connections:
- net FEED_P: now also J1.2 (Pin_2); no longer J1.1 (Pin_1)
- net GND_IN: now also J1.3 (Pin_3); no longer J1.2 (Pin_2)
- new net IGN_IN: J1.1 (Pin_1)
Changed lines of the file:
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@@
+	(wire
+		(pts
+			(xy 31.75 73.66) (xy 31.75 66.04)
+		)
+		(stroke
+			(width 0)
+			(type default)
+		)
+	)
+	(hierarchical_label "IGN_IN"
+		(shape output)
+		(at 31.75 66.04 90)
+		(effects
+			(font
+				(size 1.27 1.27)
+			)
+			(justify left)
+		)
+	)
 	(wire
 		(pts
@@
 	)
 	(symbol
-		(lib_id "Connector:Conn_01x02_Pin")
+		(lib_id "Connector:Conn_01x03_Pin")
 		(at 26.67 76.2 0)
 		(unit 1)
@@
 			)
 		)
-		(property "Value" "PWR (SS1.5 2-way)"
+		(property "Value" "PWR (SS1.5 3-way)"
 			(at 21.59 71.12 0)
 			(show_name no)
@@
 		(pin "2"
 		)
+		(pin "3"
+		)
 		(instances
