File: hardware/sheets/power_input.kicad_sch (KiCad schematic)
At the start: 31 parts, among them J1 PWR pigtail -> SS1.5 3w, Q10 IPT008N06NM5LF, Q11 IPT008N06NM5LF, Q12 MMBT3904, U10 LTC4380HMS-2

Commit message: hw(pcb): resolve D4 and U4, give GND_IN its own island, stop leaving stubs
Four things that had all been blocking a clean board, plus the pass of routing
they unblocked.

D4 is a TO-277A, whose third pad is the cathode tab.  Device:D_Schottky has no
pin 3, so schematic parity reported the tab as a net with no corresponding pin
however the pad was aliased -- aliasing pads is not a fix for a symbol that is
missing a pin.  mccan_parts:D_SCHOTTKY_TAB is that symbol with a hidden pin 3
stacked on the cathode, which is what the part actually is.

U4 was BLOCKED since Task 8 step 0 on an apparent pin-1 disagreement between two
figures of DS46371.  There is no disagreement: the Suggested Pad Layout is a bare
land pattern with no pin names, drawn in a different orientation from the Package
Outline, and the three figures that do carry pin names all agree.  Pin 1 top-left
in top view, counter-clockwise; pad 13 is the exposed pad and it is VIN, not GND.
The reasoning is written out in fpmap.py so it is not re-litigated.  fpmap's
unassignable list is now empty and says why it should stay that way.

GND_IN gets its own F.Cu island rather than sharing the pour.  GND and GND_IN are
separate nets that meet at exactly two places, L2 winding B and R3; nothing in DRC
enforces that, because a pour never shorts to a foreign net, so check_grounds.py
is the guard and it now passes: all 12 GND_IN pads inside the island, no GND pads
in it.

_ar_prune was deleting whole tracks when it should have been trimming them, and
was doing its reachability walk without regard for which layer a piece was on.
It is now layer-aware and junction-based, and trims rather than deletes.  That
takes the board from 9 dangling vias and 1 dangling track to none of either.

Also: SolderWire footprints are BOM-excluded in the library and the symbols
disagreed, which parity reported seven times over -- the footprints are right, so
in_bom() now follows them.  Silk references that collided move to F.Fab instead
of bein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
Parts:
- J1: now left out of the parts list
Changed lines of the file:
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@@
 		(body_style 1)
 		(exclude_from_sim no)
-		(in_bom yes)
+		(in_bom no)
 		(on_board yes)
 		(in_pos_files yes)

Commit message: hw(power): feed B for AUX_R, and delete the ignition sense
Co-Authored-By: Claude Sonnet 5.5 <noreply@anthropic.com>
Parts:
- added C66: 100nF, Capacitor_SMD:C_0805_2012Metric, symbol Device:C
- added D24: MMSZ5245B, Diode_SMD:D_SOD-123, symbol Device:D_Zener
- added D25: SMBJ24A, Diode_SMD:D_SMB, symbol Device:D_Zener
- added J9: SS1.5 2w feed B, Connector_Wire:SolderWire-1.5sqmm_1x02_P6mm_D1.7mm_OD3mm_Relief, symbol Connector:Conn_01x02_Pin
- added NT1: NetTie_2, NetTie:NetTie-2_SMD_Pad0.5mm, symbol Device:NetTie_2
- added Q13: SQJ461EP, Package_SO:PowerPAK_SO-8L_Single, symbol Transistor_FET:Si7141DP
- added R108: 100k, Resistor_SMD:R_0603_1608Metric, symbol Device:R
- J1: value PWR pigtail -> SS1.5 3w -> PWR feed A -> SS1.5 2w; footprint Connector_Wire:SolderWire-1.5sqmm_1x03_P6mm_D1.7mm_OD3mm_Relief -> Connector_Wire:SolderWire-1.5sqmm_1x02_P6mm_D1.7mm_OD3mm_Relief; symbol Connector:Conn_01x03_Pin -> Connector:Conn_01x02_Pin
Connections:
- net IGN_IN is gone; now on net FEED_P: J1.1 (Pin_1)
- net FEED_P: no longer J1.2 (Pin_2)
- net GND: now also NT1.2
- net GND_IN: now also J1.2 (Pin_2); no longer J1.3 (Pin_3)
- new net FEED_B_P: J9.1 (Pin_1), Q13.5 (D)
- new net GATE_B: D24.2 (A), Q13.4 (G), R108.1
- new net GND_B: C66.2, D25.2 (A), J9.2 (Pin_2), NT1.1, R108.2
- new net VBAT_B: C66.1, D24.1 (K), D25.1 (K), Q13.1 (S), Q13.2 (S), Q13.3 (S)
