File: hardware/sheets/outputs.kicad_sch (KiCad schematic)
At the start: 0 parts

Commit message: hw(sch): outputs sheet - schematic capture complete, ERC clean (Task 6)
PCA9685, 12 RGB switching channels with sense shunts, the 16:1 mux and its
sense-path protection, the dual PROFET, four PTCs and the six panel connectors.
164 symbols.  This completes schematic capture.

The gate the plan sets for this task is met: kicad-cli sch erc --severity-all
--exit-code-violations returns exit=0 with 0 errors and 0 warnings across all
five sheets.  Every unconnected pin is either connected or no-connect flagged.

ChannelIndex order verified from the netlist rather than the drawing, because
getting it wrong silently scrambles colours and corners against firmware that is
already written: LED0->PWM_FL_R through LED11->PWM_RR_B, with FET n and mux
address n lining up with PWM channel n on every one of the twelve.

Three new symbols.  ADG706 and NX5020UNBKS are verified from local datasheets;
the FET is built as a 2-unit symbol so each channel draws as one device and six
packages cover twelve channels.

Two deliberate deviations from the plan, both written up.  ~OE is pulled LOW
rather than high: taken literally the plan would leave the board permanently
dark, since no GPIO is allocated to release it, and "disabled by default" is
already delivered by the switched rail plus the PCA9685's power-on state.  And
the plan's Step 3 still quotes 1 ohm / 140 mV / 2512 shunts, which predate the
RGB load being corrected ~4x downward; the sheet is built to the current 10 ohm
/ 267 mV values.

Surfaces a cross-domain dependency that would otherwise have been lost between
disciplines: the shunt package rating is conditional on FIRMWARE latching a
shorted channel off.  Normal dissipation is 7 mW, but a shorted channel puts
~2.5 W into one shunt - ten times a 1206's rating - survivable only because the
sweep is brief and firmware stops driving it.  Recorded on the sheet, in
part-selection.md, and flagged for the firmware spec.

BLOCKER for Task 8: no Infineon datasheet for the BTS7008-2EPA is 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
Parts:
- added C41, C46: 10uF, symbol Device:C
- added C42, C43, C47: 100nF, symbol Device:C
- added C45, C48, C49, C50, C51, C52, C53, C54, C55, C56, C57, C58, C59: 10nF, symbol Device:C
- added D10, D11, D12, D13, D14, D15, D16, D17, D18, D19, D20, D21, D9: BAT54, symbol Device:D_Schottky
- added F2, F3, F4, F5: 1206L050/24, symbol Device:Polyfuse
- added J3: FL SS1.0 4w key A / black, symbol Connector:Conn_01x04_Pin
- added J4: FR SS1.0 4w key B / grey, symbol Connector:Conn_01x04_Pin
- added J5: RL SS1.0 4w key C / brown, symbol Connector:Conn_01x04_Pin
- added J6: RR SS1.0 4w key D / natural, symbol Connector:Conn_01x04_Pin
- added J7: DENALI SS1.5 3w, symbol Connector:Conn_01x03_Pin
- added J8: CAN SS1.0 2w, symbol Connector:Conn_01x02_Pin
- added Q4A, Q4B, Q5A, Q5B, Q6A, Q6B, Q7A, Q7B, Q8A, Q8B, Q9A, Q9B: NX5020UNBKS, symbol mccan_parts:NX5020UNBKS
- added R40, R41, R42, R43, R44, R45, R46, R47, R48, R49, R50, R51, R64, R65, R66, R67, R68, R69, R70, R71, R72, R73, R74, R75, R78, R79, R80: 10k, symbol Device:R
- added R52, R53, R54, R55, R56, R57, R58, R59, R60, R61, R62, R63: 10R, symbol Device:R
- added R76, R77: 4.7k, symbol Device:R
- added R81: TBD-see-note, symbol Device:R
- added R82, R83, R84, R85, R86, R87, R88, R89, R90, R91, R92, R93: 100R, symbol Device:R
- added U7: PCA9685PW, symbol Driver_LED:PCA9685PW
- added U8: ADG706, symbol mccan_parts:ADG706
- added U9: BTS7008-2EPA, symbol mccan_parts:BTS7008_2EPA
Connections:
- new net: C56.1, R90.2
- new net: C52.1, R86.2
- new net: C58.1, R92.2
- new net: C51.1, R85.2
- new net: C55.1, R89.2
- new net: C53.1, R87.2
- new net: R78.1, U7.23 (~{OE})
- new net: C50.1, R84.2
- new net: C57.1, R91.2
- new net: C59.1, R93.2
- new net: C54.1, R88.2
- new net: C48.1, R82.2
- new net: C49.1, R83.2
- new net +24V: F2.1, F3.1, F4.1, F5.1
- new net +24V_FL: F2.2, J3.1 (Pin_1)
- new net +24V_FR: F3.2, J4.1 (Pin_1)
- new net +24V_RL: F4.2, J5.1 (Pin_1)
- new net +24V_RR: F5.2, J6.1 (Pin_1)
- new net +3V3_ALW: D21.1 (K)
- new net +3V3_SW: C41.1, C42.1, C43.1, D10.1 (K), D11.1 (K), D12.1 (K), D13.1 (K), D14.1 (K), D15.1 (K), D16.1 (K), D17.1 (K), D18.1 (K), D19.1 (K), D20.1 (K), D9.1 (K), R76.2, R77.2, U7.28 (VDD), U8.1 (VDD), U8.18 (EN)
- new net CANH: J8.1 (Pin_1)
- new net CANL: J8.2 (Pin_2)
- new net DEN_A_OUT: J7.1 (Pin_1), U9.5 (OUT0)
- new net DEN_B_OUT: J7.2 (Pin_2), U9.6 (OUT1)
- new net DEN_DSEL: U9.4 (DSEL)
- new net EN_DIAG: U9.3 (DEN)
- new net GND: C41.2, C42.2, C43.2, C45.2, C46.2, C47.2, C48.2, C49.2, C50.2, C51.2, C52.2, C53.2, C54.2, C55.2, C56.2, C57.2, C58.2, C59.2, J7.3 (Pin_3), R40.2, R41.2, R42.2, R43.2, R44.2, R45.2, R46.2, R47.2, R48.2, R49.2, R50.2, R51.2, R52.2, R53.2, R54.2, R55.2, R56.2, R57.2, R58.2, R59.2, R60.2, R61.2, R62.2, R63.2, R78.2, R79.2, R80.2, R81.2, U7.1 (A0), U7.14 (VSS), U7.2 (A1), U7.24 (A5), U7.25 (EXTCLK), U7.3 (A2), U7.4 (A3), U7.5 (A4), U8.12 (GND), U8.27 (VSS), U8.4 (S16), U8.5 (S15), U8.6 (S14), U8.7 (S13), U9.9 (GND)
- new net I2C_SCL: R77.1, U7.26 (SCL)
- new net I2C_SDA: R76.1, U7.27 (SDA)
- new net ISNS_DEN: D21.2 (A), R81.1, U9.7 (IS)
- new net MUXIN_FL_B: D11.2 (A), R66.2, U8.21 (S3)
- new net MUXIN_FL_G: D10.2 (A), R65.2, U8.20 (S2)
- new net MUXIN_FL_R: D9.2 (A), R64.2, U8.19 (S1)
- new net MUXIN_FR_B: D14.2 (A), R69.2, U8.24 (S6)
- new net MUXIN_FR_G: D13.2 (A), R68.2, U8.23 (S5)
- new net MUXIN_FR_R: D12.2 (A), R67.2, U8.22 (S4)
- new net MUXIN_RL_B: D17.2 (A), R72.2, U8.11 (S9)
- new net MUXIN_RL_G: D16.2 (A), R71.2, U8.26 (S8)
- new net MUXIN_RL_R: D15.2 (A), R70.2, U8.25 (S7)
- new net MUXIN_RR_B: D20.2 (A), R75.2, U8.8 (S12)
- new net MUXIN_RR_G: D19.2 (A), R74.2, U8.9 (S11)
- new net MUXIN_RR_R: D18.2 (A), R73.2, U8.10 (S10)
- new net MUX_S0: U8.17 (A0)
- new net MUX_S1: U8.16 (A1)
- new net MUX_S2: U8.15 (A2)
- new net MUX_S3: U8.14 (A3)
- new net PWM_DEN_A: R79.1, U9.1 (IN0)
- new net PWM_DEN_B: R80.1, U9.2 (IN1)
- new net PWM_FL_B: Q5A.2 (G1), R42.1, U7.8 (LED2)
- new net PWM_FL_G: Q4B.5 (G2), R41.1, U7.7 (LED1)
- new net PWM_FL_R: Q4A.2 (G1), R40.1, U7.6 (LED0)
- new net PWM_FR_B: Q6B.5 (G2), R45.1, U7.11 (LED5)
- new net PWM_FR_G: Q6A.2 (G1), R44.1, U7.10 (LED4)
- new net PWM_FR_R: Q5B.5 (G2), R43.1, U7.9 (LED3)
- new net PWM_RL_B: Q8A.2 (G1), R48.1, U7.15 (LED8)
- new net PWM_RL_G: Q7B.5 (G2), R47.1, U7.13 (LED7)
- new net PWM_RL_R: Q7A.2 (G1), R46.1, U7.12 (LED6)
- new net PWM_RR_B: Q9B.5 (G2), R51.1, U7.18 (LED11)
- new net PWM_RR_G: Q9A.2 (G1), R50.1, U7.17 (LED10)
- new net PWM_RR_R: Q8B.5 (G2), R49.1, U7.16 (LED9)
- new net RET_FL_B: J3.4 (Pin_4), Q5A.6 (D1), R84.1
- new net RET_FL_G: J3.3 (Pin_3), Q4B.3 (D2), R83.1
- new net RET_FL_R: J3.2 (Pin_2), Q4A.6 (D1), R82.1
- new net RET_FR_B: J4.4 (Pin_4), Q6B.3 (D2), R87.1
- new net RET_FR_G: J4.3 (Pin_3), Q6A.6 (D1), R86.1
- new net RET_FR_R: J4.2 (Pin_2), Q5B.3 (D2), R85.1
- new net RET_RL_B: J5.4 (Pin_4), Q8A.6 (D1), R90.1
- new net RET_RL_G: J5.3 (Pin_3), Q7B.3 (D2), R89.1
- new net RET_RL_R: J5.2 (Pin_2), Q7A.6 (D1), R88.1
- new net RET_RR_B: J6.4 (Pin_4), Q9B.3 (D2), R93.1
- new net RET_RR_G: J6.3 (Pin_3), Q9A.6 (D1), R92.1
- new net RET_RR_R: J6.2 (Pin_2), Q8B.3 (D2), R91.1
- new net RGB_ISNS: C45.1, U8.28 (D)
- new net SENSE_FL_B: Q5A.1 (S1), R54.1, R66.1
- new net SENSE_FL_G: Q4B.4 (S2), R53.1, R65.1
- new net SENSE_FL_R: Q4A.1 (S1), R52.1, R64.1
- new net SENSE_FR_B: Q6B.4 (S2), R57.1, R69.1
- new net SENSE_FR_G: Q6A.1 (S1), R56.1, R68.1
- new net SENSE_FR_R: Q5B.4 (S2), R55.1, R67.1
- new net SENSE_RL_B: Q8A.1 (S1), R60.1, R72.1
- new net SENSE_RL_G: Q7B.4 (S2), R59.1, R71.1
- new net SENSE_RL_R: Q7A.1 (S1), R58.1, R70.1
- new net SENSE_RR_B: Q9B.4 (S2), R63.1, R75.1
- new net SENSE_RR_G: Q9A.1 (S1), R62.1, R74.1
- new net SENSE_RR_R: Q8B.4 (S2), R61.1, R73.1
- new net VBAT: C46.1, C47.1, U9.8 (VS)
- no-connect marks 0 -> 7

Commit message: hw(sch): PROFET verified against the real datasheet, Task 8 unblocked
The Infineon BTS7008-2EPA datasheet (Rev. 1.21, 2024-07-29) arrived, so U9's
placeholder pinout could finally be checked. It was wrong in every position.

Table 2 p.6: VS is the EXPOSED PAD -- there is no side supply pin at all -- and
each output is three pins (8-10 OUT1, 12-14 OUT0) that note 1 requires to be
tied together and to carry the full channel current. Pins 7 and 11 are not
bonded. Six pins that did not exist in the placeholder exist in the part.

R81 is sized: kILIS = 5400 at 2.8 A, so the Denali's 3.3 A gives 611 uA at IS,
and 2.2k puts that at 1.34 V -- mid-scale for ADC1 at 11 dB, full scale at
6.0 A, floor at 368 mA against a ~21 mA open-load current.

Reading the datasheet also found a real defect in the Task 6 sheet: under fault
the IS pin saturates (IIS(SAT) 4.1-15 mA, VS - VIS only 0.5 V typ / 1 V max),
so the sense node reaches ~12.5 V, and that node was wired to GPIO 34 through
nothing but a Schottky clamp. Added R82/R83 (RIS_PROT, RADC) per Figure 43,
with C47 (CSENSE) and C48 at the ADC. Firmware must settle >= 250 us after a
DSEL change.

Added the Table 24 series resistors on the four control lines, which are what
lets the outputs switch OFF on loss of ground. Their pulldowns go on the MCU
side: in series they would divide 3.3 V down to 2.24 V against a 2.0 V max
guaranteed-high threshold. EN_DIAG and DEN_DSEL keep R35/R34 from mcu_can's
passive-defaults block rather than being duplicated here.

Footprint identified: Package_SO:Infineon_PG-TSDSO-14-22 ships with KiCad and
numbers the thermal pad 15, which is why VS is pin 15. Also closed a
pre-existing C44 gap, so designators are now gapless in every series.

ERC --severity-all --exit-code-violations: exit=0, 0 errors, 0 warnings.
166 nets, every PROFET net read back from the netlist. ChannelIndex unchanged.

Co-Authored-By: Claude Opus 5 <noreply@anthropic.com>
Claude-Session: https://claude.ai/code/session_01Bkq7QP4he4cd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
Parts:
- added C44, C60: 10nF, symbol Device:C
- added R94, R95, R96, R97, R98, R99: 100R, symbol Device:R
- C45: value 10nF -> 10uF
- C46: value 10uF -> 100nF
- C47: value 100nF -> 220pF
- C48: now fitted
- R79, R80: value 10k -> 4.7k
- R81: value TBD-see-note -> 2.2k
- R82, R83, R84, R85: value 100R -> 4.7k; now fitted
- R86, R87: value 100R -> 10k; now fitted
Connections:
- net DEN_A_OUT: now also U9.12 (OUT0), U9.13 (OUT0), U9.14 (OUT0); no longer U9.5 (OUT0)
- net DEN_B_OUT: now also U9.10 (OUT1), U9.8 (OUT1), U9.9 (OUT1); no longer U9.6 (OUT1)
- net DEN_DSEL: now also R85.1; no longer U9.4 (DSEL)
- net EN_DIAG: now also R84.1; no longer U9.3 (DEN)
- net GND: now also R86.2, R87.2, U9.1 (GND), C44.2, C60.2; no longer R79.2, R80.2, U9.9 (GND)
- net ISNS_DEN: now also C48.1, R83.2; no longer R81.1, U9.7 (IS)
- net PWM_DEN_A: now also R86.1; no longer U9.1 (IN0)
- net PWM_DEN_B: now also R87.1; no longer U9.2 (IN1)
- net RET_FL_B: now also R90.1; no longer R84.1
- net RET_FL_G: now also R89.1; no longer R83.1
- net RET_FL_R: now also R88.1; no longer R82.1
- net RET_FR_B: now also R93.1; no longer R87.1
- net RET_FR_G: now also R92.1; no longer R86.1
- net RET_FR_R: now also R91.1; no longer R85.1
- net RET_RL_B: now also R96.1; no longer R90.1
- net RET_RL_G: now also R95.1; no longer R89.1
- net RET_RL_R: now also R94.1; no longer R88.1
- net RET_RR_B: now also R99.1; no longer R93.1
- net RET_RR_G: now also R98.1; no longer R92.1
- net RET_RR_R: now also R97.1; no longer R91.1
- net RGB_ISNS: now also C44.1; no longer C45.1
- net VBAT: now also C45.1, U9.15 (VS); no longer C47.1, U9.8 (VS)
- net at R90.2: now also C51.1; no longer C56.1
- net at C52.1: now also R91.2; no longer R86.2
- net at R92.2: now also C53.1; no longer C58.1
- net at R85.2: now also U9.5 (DSEL); no longer C51.1
- net at R89.2: now also C50.1; no longer C55.1
- net at R84.2: now also U9.3 (DEN); no longer C50.1
- net at C57.1: now also R96.2; no longer R91.2
- net at C59.1: now also R98.2; no longer R93.2
- net at C54.1: now also R93.2; no longer R88.2
- net at R82.2: now also C47.1, R81.1, R83.1; no longer C48.1
- net at C49.1: now also R88.2; no longer R83.2
- new net: C60.1, R99.2
- new net: C55.1, R94.2
- new net: C58.1, R97.2
- new net: R79.2, U9.2 (IN0)
- new net: R82.1, U9.4 (IS)
- new net: R80.2, U9.6 (IN1)
- new net: C56.1, R95.2
- no-connect marks 7 -> 9
Other:
- moved on the sheet: C45, C46, C47, C49, C50, C51, C52, C53, C54, C55, C56, C57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

Commit message: hw(sch): sweep every selected part into the schematic; D6+D7 become one PESD2CANFD24U-T
Closes the gap the Task 7 review's finding F1 was about: parts chosen in
prose had not reached the generators, which is exactly how the superseded
SQJ415EP survived five days in the schematic.

STRUCTURAL - the CAN ESD pair is now one part. D6 and D7 were two placeholder
"24V bidir" discretes; the Nexperia PESD2CANFD24U-T is a single SOT23 holding
both bidirectional elements (K1/K2/CC). New verified symbol in symlib.py built
from Table 2 of the datasheet, added to gen_mcu_can's lib_symbols, and
Device:D_TVS dropped from that sheet since D6/D7 were its only users.

The two protected pins land exactly on the CANH and CANL runs, so each run is
drawn as TWO segments meeting AT the pin rather than one segment the pin
happens to touch. A pin sitting mid-wire does connect, but this project has
already produced one silent connectivity defect of that shape (labels
mid-wire, 14 instances), so the pin is made a wire endpoint and junctioned.
Verified from the netlist rather than from ERC: D6.1 -> /CANH, D6.2 -> /CANL,
D6.3 -> GND.

Consolidating freed D7, so the diode series was renumbered to stay gapless:
the ignition-divider BAT54 D8 -> D7, the twelve RGB sense clamps D9-D20 ->
D8-D19, and the PROFET sense clamp D21 -> D20. Every designator series is
gapless: C1-61, D1-20, F1-5, J1-8, L1-6, Q1-9, R1-99, SW1-2, U1-9.

VALUE SWEEP - L4/L5 "22uH" -> XAL7070-223ME, L6 "51uH CM choke" ->
ACT45B-510-2P-TL003, C3 "220uF" -> "220uF 63V" (the SMBJ24A's 8/20 us clamp is
50.6 V, so a 50 V part has no margin), U7 -> PCA9685PW/Q900, the only
AEC-Q100 variant in the ordering table. U7's lib_id stays Driver_LED:PCA9685PW
- that is the stock symbol's name, and the package is the same TSSOP28. D4 was
already SS5PH102.

FOOTPRINT - installed the vendor SamacSys footprint and STEP model for the
Wurth choke as footprints/mccan.pretty/Wurth_WE-CMBNC_7448031002.kicad_mod and
3dmodels/. Its pads verify against t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
Parts:
- removed D21: BAT54, symbol Device:D_Schottky
- added D8: BAT54, symbol Device:D_Schottky
- U7: value PCA9685PW -> PCA9685PW/Q900
Connections:
- net +3V3_ALW: now also D20.1 (K)
- net +3V3_SW: now also D8.1 (K); no longer D20.1 (K)
- net ISNS_DEN: now also D20.2 (A)
- net MUXIN_FL_B: now also D10.2 (A); no longer D11.2 (A)
- net MUXIN_FL_G: now also D9.2 (A); no longer D10.2 (A)
- net MUXIN_FL_R: now also D8.2 (A); no longer D9.2 (A)
- net MUXIN_FR_B: now also D13.2 (A); no longer D14.2 (A)
- net MUXIN_FR_G: now also D12.2 (A); no longer D13.2 (A)
- net MUXIN_FR_R: now also D11.2 (A); no longer D12.2 (A)
- net MUXIN_RL_B: now also D16.2 (A); no longer D17.2 (A)
- net MUXIN_RL_G: now also D15.2 (A); no longer D16.2 (A)
- net MUXIN_RL_R: now also D14.2 (A); no longer D15.2 (A)
- net MUXIN_RR_B: now also D19.2 (A); no longer D20.2 (A)
- net MUXIN_RR_G: now also D18.2 (A); no longer D19.2 (A)
- net MUXIN_RR_R: now also D17.2 (A); no longer D18.2 (A)
Other:
- moved on the sheet: D10, D11, D12, D13, D14, D15, D16, D17, D18, D19, D20, D9

Commit message: hw(pcb): Task 8 step 0 - footprints assigned, 209 of 219 verified
Nothing in the project had a footprint except the PROFET's. Assignment now
lives in one auditable place, scripts/fpmap.py, which the four sheet
generators call when emitting each symbol's Footprint property. No generator
chooses a footprint of its own any more.

Three rules, and the reasoning is in the file rather than in a commit nobody
will read again: signal passives are 0603; a passive gets a bigger package
only for a stated reason; and nothing gets a footprint that has not been
checked to exist.

The reasons that drove a larger package:
- R2/R3, the 0R links bypassing the input choke windings, are 2512. They are
  DNP, but if anyone fits them for the tied-ground prototype they carry the
  entire 7.0 A night load, and a 0603 link is rated about 1 A.
- R52-R63, the RGB sense shunts, are 1206 for the FAULT case, not the normal
  7 mW. The package is sized on the understanding that firmware latches a
  shorted channel off; if that is ever dropped they must become 2512 1 W.
- The front-end ceramics are sized against the SMBJ24A's 8/20 us clamp of
  50.6 V, not the 38.9 V the distributor summaries quote. 100 nF fits 0805 at
  100 V; 1-2.2 uF at 63 V does not fit 0805; 10 uF at 63 V needs 1210.
- C20-C22 on +24 V are 1206 for DC-BIAS derating, a different reason - a 25 V
  X7R at 24 V keeps only 40-60% of nameplate.

Package identifications read from the datasheets rather than assumed:
NX5020UNBKS is SOT363/SC-88 (section 1), LM51571-Q1 RTE is WQFN-16 3x3 with a
1.66 mm exposed pad (so KiCad's EP1.675x1.675 is within tolerance), SS5PH102
is TO-277A, PESD2CANFD24U-T is SOT23.

FLAGGED, not silently accepted: the LM5164 DDA thermal pad is 3.4 x 2.8 mm on
the mechanical drawing and KiCad has no exact match. EP2.62x3.51 is the
closest by area (9.20 mm2 against 9.52) and is used for now, but that pad is
the part's heatsink on a thermally critical rail, so an exact DDA land pattern
should be drawn before fabr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
Parts:
- C41, C42, C43, C44, C47, C48: footprint (none) -> Capacitor_SMD:C_0603_1608Metric
- C45: footprint (none) -> Capacitor_SMD:C_1210_3225Metric
- C46: footprint (none) -> Capacitor_SMD:C_0805_2012Metric
- C49, C50, C51, C52, C53, C54, C55, C56, C57, C58, C59, C60: footprint (none) -> Capacitor_SMD:C_1206_3216Metric
- D10, D11, D12, D13, D14, D15, D16, D17, D18, D19, D20, D8, D9: footprint (none) -> Diode_SMD:D_SOD-123
- F2, F3, F4, F5: footprint (none) -> Fuse:Fuse_1206_3216Metric
- Q4A, Q4B, Q5A, Q5B, Q6A, Q6B, Q7A, Q7B, Q8A, Q8B, Q9A, Q9B: footprint (none) -> Package_TO_SOT_SMD:SOT-363_SC-70-6
- R40, R41, R42, R43, R44, R45, R46, R47, R48, R49, R50, R51, R64, R65, R66, R67, R68, R69, R70, R71, R72, R73, R74, R75, R76, R77, R78, R79, R80, R81, R82, R83, R84, R85, R86, R87: footprint (none) -> Resistor_SMD:R_0603_1608Metric
- R52, R53, R54, R55, R56, R57, R58, R59, R60, R61, R62, R63, R88, R89, R90, R91, R92, R93, R94, R95, R96, R97, R98, R99: footprint (none) -> Resistor_SMD:R_1206_3216Metric
- U7, U8: footprint (none) -> Package_SO:TSSOP-28_4.4x9.7mm_P0.65mm
- U9: footprint (none) -> Package_SO:Infineon_PG-TSDSO-14-22

Commit message: hw(sch): CM chokes were wired to KiCad's pin numbering, not the parts'
Both common-mode chokes used Device:L_Coupled, which numbers its pins
winding A = 1-2, winding B = 3-4.  Every real four-terminal CM choke numbers
them winding A = 1-4, winding B = 2-3.  Both parts in this design are real
ones, so both were wired across the wrong pairs.

L2 was the serious one.  As drawn, winding 1-4 tied VBAT_PROT to board GND
and winding 2-3 tied VBAT_F to GND_IN -- two dead shorts across the supply
through 6.3 mOhm windings.  First power-up would have cleared the 10 A fuse
with the P-FET and the choke carrying the fault.

L6 transposed CANH and CANL between the transceiver and the connector, so the
board would never have received a frame.  Being listen-only by default, the
symptom is "no traffic" -- which spec 8.3 already names as the top risk and
the thing most likely to be misdiagnosed as a firmware fault.

ERC passes either way.  DRC passes either way.  The footprint pad count
matches either way.  Nothing automated catches this.

Verified from the VECTOR GEOMETRY of both datasheets, not a text dump -- a
flat extraction gives four bare numerals with no axis:
  Wurth WE-CMBNC 7448031002 "Schematic": upper coil's leads sit under labels
    1 (x=347.0) and 4 (x=488.6); lower coil's under 2 and 3 at the same x.
  TDK ACT45B "CIRCUIT DIAGRAM": identical, 1/4 upper, 2/3 lower.

Fix is a mccan_parts:CM_CHOKE_4T symbol drawn with L_Coupled's own graphics
but numbered to match the parts.  Not one wire moves -- which is also why the
drawing never looked wrong.  Netlist now reads:
  L2.1->4  VBAT_PROT -> VBAT_F      L2.2->3  GND_IN -> GND
  L6.1->4  U6 CANH   -> CANH        L6.2->3  U6 CANL -> CANL

Also in this commit, from the two datasheets supplied today:

- Superseal is a WIRE-TO-WIRE series with no panel-mount board-side housing,
  so the seven "panel connectors" could never have been built, and that is
  why all seven sat in fpmap.BLOCKED through Task 8 step 0.  J1 and J3-J8
  b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
Parts:
- J3: value FL SS1.0 4w key A / black -> FL pigtail -> SS1.0 key A / black; footprint (none) -> Connector_Wire:SolderWire-0.5sqmm_1x04_P4.6mm_D0.9mm_OD2.1mm_Relief
- J4: value FR SS1.0 4w key B / grey -> FR pigtail -> SS1.0 key B / grey; footprint (none) -> Connector_Wire:SolderWire-0.5sqmm_1x04_P4.6mm_D0.9mm_OD2.1mm_Relief
- J5: value RL SS1.0 4w key C / brown -> RL pigtail -> SS1.0 key C / brown; footprint (none) -> Connector_Wire:SolderWire-0.5sqmm_1x04_P4.6mm_D0.9mm_OD2.1mm_Relief
- J6: value RR SS1.0 4w key D / natural -> RR pigtail -> SS1.0 key D / natural; footprint (none) -> Connector_Wire:SolderWire-0.5sqmm_1x04_P4.6mm_D0.9mm_OD2.1mm_Relief
- J7: value DENALI SS1.5 3w -> DENALI pigtail -> SS1.5 3w; footprint (none) -> Connector_Wire:SolderWire-1.5sqmm_1x03_P6mm_D1.7mm_OD3mm_Relief
- J8: value CAN SS1.0 2w -> CAN pigtail -> SS1.0 2w; footprint (none) -> Connector_Wire:SolderWire-0.5sqmm_1x02_P4.6mm_D0.9mm_OD2.1mm_Relief
