File: hardware/sheets/outputs.kicad_sch (KiCad schematic)
At the start: 118 parts, among them J3 FL pigtail -> SS1.0 key A / b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, J4 FR pigtail -> SS1.0 key B / g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, J5 RL pigtail -> SS1.0 key C / b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, J6 RR pigtail -> SS1.0 key D / n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, J7 DENALI pigtail -> SS1.5 3w, J8 CAN pigtail -> SS1.0 2w, Q4A NX5020UNBKS, Q4B NX5020UNBKS, Q5A NX5020UNBKS, Q5B NX5020UNBKS, Q6A NX5020UNBKS, Q6B NX5020UNBKS, Q7A NX5020UNBKS, Q7B NX5020UNBKS, Q8A NX5020UNBKS, Q8B NX5020UNBKS, Q9A NX5020UNBKS, Q9B NX5020UNBKS, U7 PCA9685PW/Q900, U8 ADG706, U9 BTS7008-2EPA

Commit message: hw(pcb): resolve D4 and U4, give GND_IN its own island, stop leaving stubs
Four things that had all been blocking a clean board, plus the pass of routing
they unblocked.

D4 is a TO-277A, whose third pad is the cathode tab.  Device:D_Schottky has no
pin 3, so schematic parity reported the tab as a net with no corresponding pin
however the pad was aliased -- aliasing pads is not a fix for a symbol that is
missing a pin.  mccan_parts:D_SCHOTTKY_TAB is that symbol with a hidden pin 3
stacked on the cathode, which is what the part actually is.

U4 was BLOCKED since Task 8 step 0 on an apparent pin-1 disagreement between two
figures of DS46371.  There is no disagreement: the Suggested Pad Layout is a bare
land pattern with no pin names, drawn in a different orientation from the Package
Outline, and the three figures that do carry pin names all agree.  Pin 1 top-left
in top view, counter-clockwise; pad 13 is the exposed pad and it is VIN, not GND.
The reasoning is written out in fpmap.py so it is not re-litigated.  fpmap's
unassignable list is now empty and says why it should stay that way.

GND_IN gets its own F.Cu island rather than sharing the pour.  GND and GND_IN are
separate nets that meet at exactly two places, L2 winding B and R3; nothing in DRC
enforces that, because a pour never shorts to a foreign net, so check_grounds.py
is the guard and it now passes: all 12 GND_IN pads inside the island, no GND pads
in it.

_ar_prune was deleting whole tracks when it should have been trimming them, and
was doing its reachability walk without regard for which layer a piece was on.
It is now layer-aware and junction-based, and trims rather than deletes.  That
takes the board from 9 dangling vias and 1 dangling track to none of either.

Also: SolderWire footprints are BOM-excluded in the library and the symbols
disagreed, which parity reported seven times over -- the footprints are right, so
in_bom() now follows them.  Silk references that collided move to F.Fab instead
of bein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
Parts:
- J3, J4, J5, J6, J7, J8: now left out of the parts list
Changed lines of the file:
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@@
 		(body_style 1)
 		(exclude_from_sim no)
-		(in_bom yes)
+		(in_bom no)
 		(on_board yes)
 		(in_pos_files yes)
@@
 		(body_style 1)
 		(exclude_from_sim no)
-		(in_bom yes)
+		(in_bom no)
 		(on_board yes)
 		(in_pos_files yes)
@@
 		(body_style 1)
 		(exclude_from_sim no)
-		(in_bom yes)
+		(in_bom no)
 		(on_board yes)
 		(in_pos_files yes)
@@
 		(body_style 1)
 		(exclude_from_sim no)
-		(in_bom yes)
+		(in_bom no)
 		(on_board yes)
 		(in_pos_files yes)
@@
 		(body_style 1)
 		(exclude_from_sim no)
-		(in_bom yes)
+		(in_bom no)
 		(on_board yes)
 		(in_pos_files yes)
@@
 		(body_style 1)
 		(exclude_from_sim no)
-		(in_bom yes)
+		(in_bom no)
 		(on_board yes)
 		(in_pos_files yes)

Commit message: hw(outputs): ten signal channels on three quad smart high-side switches
Replace the plan3 RGB/PWM stage (PCA9685, ADG706, NX5020 channels and
shunts, DNP snubbers, BTS7008, PTCs, J6, J7) with U11-U13 TPS4H160B-Q1
per D1: 4.7k series + 47k pull-down on every IN, CS -> 1.8k + 4.7k ->
SNS_x with the BAT54 clamp on the ADC side only, R_CL, R_THER to +5V,
C_VS 100nF 100V 0805, FAULT/NC no-connect. Harness tails J3/J4/J5 per
D5; J8 (CAN) unchanged. OUT_AUX_L/R end in one 47k pull-down each.

Co-Authored-By: Claude Opus 5.5 <noreply@anthropic.com>
Parts:
- removed C47: 220pF, Capacitor_SMD:C_0603_1608Metric, symbol Device:C
- removed C48: 10nF, Capacitor_SMD:C_0603_1608Metric, symbol Device:C
- removed C49, C50, C51, C52, C53, C54, C55, C56, C57, C58, C59, C60: 10nF, Capacitor_SMD:C_1206_3216Metric, symbol Device:C
- removed D11, D12, D13, D14, D15, D16, D17, D18, D19, D20: BAT54, Diode_SMD:D_SOD-123, symbol Device:D_Schottky
- removed F2, F3, F4, F5: 1206L050/24, Fuse:Fuse_1206_3216Metric, symbol Device:Polyfuse
- removed J6: RR pigtail -> SS1.0 key D / natural, Connector_Wire:SolderWire-0.5sqmm_1x04_P4.6mm_D0.9mm_OD2.1mm_Relief, symbol Connector:Conn_01x04_Pin
- removed J7: DENALI pigtail -> SS1.5 3w, Connector_Wire:SolderWire-1.5sqmm_1x03_P6mm_D1.7mm_OD3mm_Relief, symbol Connector:Conn_01x03_Pin
- removed Q4A, Q4B, Q5A, Q5B, Q6A, Q6B, Q7A, Q7B, Q8A, Q8B, Q9A, Q9B: NX5020UNBKS, Package_TO_SOT_SMD:SOT-363_SC-70-6, symbol mccan_parts:NX5020UNBKS
- removed R76, R77, R79, R80, R82, R83, R84, R85: 4.7k, Resistor_SMD:R_0603_1608Metric, symbol Device:R
- removed R78, R86, R87: 10k, Resistor_SMD:R_0603_1608Metric, symbol Device:R
- removed R81: 2.2k, Resistor_SMD:R_0603_1608Metric, symbol Device:R
- removed R88, R89, R90, R91, R92, R93, R94, R95, R96, R97, R98, R99: 100R, Resistor_SMD:R_1206_3216Metric, symbol Device:R
- removed U7: PCA9685PW/Q900, Package_SO:TSSOP-28_4.4x9.7mm_P0.65mm, symbol Driver_LED:PCA9685PW
- removed U8: ADG706, Package_SO:TSSOP-28_4.4x9.7mm_P0.65mm, symbol mccan_parts:ADG706
- removed U9: BTS7008-2EPA, Package_SO:Infineon_PG-TSDSO-14-22, symbol mccan_parts:BTS7008_2EPA
- added U11, U12, U13: TPS4H160BQPWPRQ1, Package_SO:HTSSOP-28-1EP_4.4x9.7mm_P0.65mm_EP2.85x5.4mm, symbol mccan_parts:TPS4H160B_Q1
- C41: value 10uF -> 100nF 100V; footprint Capacitor_SMD:C_0603_1608Metric -> Capacitor_SMD:C_0805_2012Metric
- C42, C43: value 100nF -> 100nF 100V; footprint Capacitor_SMD:C_0603_1608Metric -> Capacitor_SMD:C_0805_2012Metric
- C45: value 10uF -> 10nF; footprint Capacitor_SMD:C_1210_3225Metric -> Capacitor_SMD:C_0603_1608Metric
- C46: value 100nF -> 10nF; footprint Capacitor_SMD:C_0805_2012Metric -> Capacitor_SMD:C_0603_1608Metric
- J3: value FL pigtail -> SS1.0 key A / black -> FRONT tail; footprint Connector_Wire:SolderWire-0.5sqmm_1x04_P4.6mm_D0.9mm_OD2.1mm_Relief -> Connector_Wire:SolderWire-0.5sqmm_1x05_P4.6mm_D0.9mm_OD2.1mm_Relief; symbol Connector:Conn_01x04_Pin -> Connector:Conn_01x05_Pin
- J4: value FR pigtail -> SS1.0 key B / grey -> REAR tail 1 (7-core)
- J5: value RL pigtail -> SS1.0 key C / brown -> REAR tail 2 (7-core); footprint Connector_Wire:SolderWire-0.5sqmm_1x04_P4.6mm_D0.9mm_OD2.1mm_Relief -> Connector_Wire:SolderWire-0.5sqmm_1x03_P4.6mm_D0.9mm_OD2.1mm_Relief; symbol Connector:Conn_01x04_Pin -> Connector:Conn_01x03_Pin
- R40, R41, R42, R43, R44, R45, R46, R47, R48, R49, R71, R72, R73: value 10k -> 4.7k
- R50, R51, R74, R75: value 10k -> 47k
- R52, R53, R54, R55, R56, R57, R58, R59, R60, R61: value 10R -> 47k; footprint Resistor_SMD:R_1206_3216Metric -> Resistor_SMD:R_0603_1608Metric
- R62, R63: value 10R -> 4.02k; footprint Resistor_SMD:R_1206_3216Metric -> Resistor_SMD:R_0603_1608Metric
- R64: value 10k -> 4.02k
- R68, R69, R70: value 10k -> 1.8k
Connections:
- net MUXIN_FR_B is gone; now on net GND: R69.2
- net MUXIN_FR_G is gone; now on net GND: R68.2
- net MUXIN_RL_B is gone; now on net SNS_B: R72.2
- net MUXIN_RL_G is gone; now on net SNS_A: R71.2
- net MUXIN_RL_R is gone; now on net GND: R70.2
- net MUXIN_RR_B is gone; now on net GND: R75.2
- net MUXIN_RR_G is gone; now on net GND: R74.2
- net MUXIN_RR_R is gone; now on net SNS_C: R73.2
- net RET_FR_B is gone; now on net GND: J4.4 (Pin_4)
- net RGB_ISNS is gone; now on net SNS_A: C44.1
- net +3V3_ALW: now also D10.1 (K), D8.1 (K), D9.1 (K)
- net GND: now also J3.5 (Pin_5), R64.2, U11.1 (GND), U11.12 (GND), U11.29 (EP), U12.1 (GND), U12.12 (GND), U12.29 (EP), U13.1 (GND), U13.12 (GND), U13.29 (EP); no longer R40.2, R41.2, R42.2, R43.2, R44.2, R45.2, R46.2, R47.2, R48.2, R49.2
- net VBAT: now also C41.1, C42.1, C43.1, U11.20 (VS), U11.21 (VS), U11.22 (VS), U11.23 (VS), U12.20 (VS), U12.21 (VS), U12.22 (VS), U12.23 (VS), U13.20 (VS), U13.21 (VS), U13.22 (VS), U13.23 (VS); no longer C45.1, C46.1
- net +24V_FL renamed FL_DRL
- net FL_DRL: now also U11.27 (OUT1), U11.28 (OUT1)
- net +24V_FR renamed RL_DRL
- net RL_DRL: now also U11.17 (OUT3), U11.18 (OUT3)
- net +24V_RL renamed RR_DRL
- net RR_DRL: now also U12.17 (OUT3), U12.18 (OUT3)
- removed net +3V3_SW: C41.1, C42.1, C43.1, D10.1 (K), D8.1 (K), D9.1 (K)
- net MUXIN_FL_B renamed SNS_C
- net SNS_C: now also C46.1; no longer R66.2
- net MUXIN_FL_G renamed SNS_B
- net SNS_B: now also C45.1; no longer R65.2
- net MUXIN_FL_R renamed SNS_A
- net SNS_A: no longer R64.2
- net MUXIN_FR_R renamed THER_C
- net THER_C: now also U13.13 (THER)
- net PWM_FL_B renamed OUT_RL_DRL
- net PWM_FL_G renamed OUT_FL_IND
- net PWM_FL_R renamed OUT_FL_DRL
- net PWM_FR_B renamed OUT_FR_IND
- net PWM_FR_G renamed OUT_FR_DRL
- net PWM_FR_R renamed OUT_RL_IND
- net PWM_RL_B renamed OUT_RL_BRK
- net PWM_RL_G renamed OUT_RR_IND
- net PWM_RL_R renamed OUT_RR_DRL
- net PWM_RR_B renamed IN_FL_IND
- net IN_FL_IND: now also R41.2, U11.4 (IN2)
- net PWM_RR_G renamed IN_FL_DRL
- net IN_FL_DRL: now also R40.2, U11.3 (IN1)
- net PWM_RR_R renamed OUT_RR_BRK
- net RET_FL_B renamed FR_IND
- net FR_IND: now also U12.25 (OUT2), U12.26 (OUT2)
- net RET_FL_G renamed FR_DRL
- net FR_DRL: now also U12.27 (OUT1), U12.28 (OUT1)
- net RET_FL_R renamed FL_IND
- net FL_IND: now also U11.25 (OUT2), U11.26 (OUT2)
- net RET_FR_G renamed RL_BRK
- net RL_BRK: now also U13.27 (OUT1), U13.28 (OUT1)
- net RET_FR_R renamed RL_IND
- net RL_IND: now also U11.15 (OUT4), U11.16 (OUT4)
- removed net RET_RL_B: J5.4 (Pin_4)
- net RET_RL_G renamed RR_BRK
- net RR_BRK: now also U13.25 (OUT2), U13.26 (OUT2)
- net RET_RL_R renamed RR_IND
- net RR_IND: now also U12.15 (OUT4), U12.16 (OUT4)
- net SENSE_FL_B renamed +5V
- net +5V: now also R65.1, R67.1; no longer R54.1
- net SENSE_FL_G renamed IN_RL_IND
- net IN_RL_IND: now also R43.2, U11.6 (IN4); no longer R65.1
- net SENSE_FL_R renamed CL_C
- net CL_C: now also U13.11 (CL); no longer R52.1
- net SENSE_FR_B renamed CS_B
- net CS_B: now also R72.1, U12.10 (SNS); no longer R57.1
- net SENSE_FR_G renamed CS_A
- net CS_A: now also R71.1, U11.10 (SNS); no longer R56.1
- net SENSE_FR_R renamed IN_FR_IND
- net IN_FR_IND: now also R45.2, U12.4 (IN2); no longer R67.1
- net SENSE_RL_B renamed IN_U13_CH3_SPARE
- net IN_U13_CH3_SPARE: now also U13.5 (IN3); no longer R72.1
- net SENSE_RL_G renamed IN_RR_BRK
- net IN_RR_BRK: now also R49.2, U13.4 (IN2); no longer R71.1
- net SENSE_RL_R renamed CS_C
- net CS_C: now also R73.1, U13.10 (SNS); no longer R58.1
- net SENSE_RR_B renamed CL_B
- net CL_B: now also U12.11 (CL); no longer R75.1
- net SENSE_RR_G renamed CL_A
- net CL_A: now also U11.11 (CL); no longer R74.1
- net SENSE_RR_R renamed IN_U13_CH4_SPARE
- net IN_U13_CH4_SPARE: now also U13.6 (IN4); no longer R73.1
- new net DIAG_EN_Q: U11.14 (DIAG_EN), U12.14 (DIAG_EN), U13.14 (DIAG_EN)
- new net DIAG_SEL0_Q: U11.8 (SEL0), U12.8 (SEL0), U13.8 (SEL0)
- new net DIAG_SEL1_Q: U11.7 (SEL1), U12.7 (SEL1), U13.7 (SEL1)
- new net IN_FR_DRL: R44.2, R54.1, U12.3 (IN1)
- new net IN_RL_BRK: R48.2, R58.1, U13.3 (IN1)
- new net IN_RL_DRL: R42.2, R52.1, U11.5 (IN3)
- new net IN_RR_DRL: R46.2, R56.1, U12.5 (IN3)
- new net IN_RR_IND: R47.2, R57.1, U12.6 (IN4)
- new net OUT_AUX_L: R74.1
- new net OUT_AUX_R: R75.1
- new net THER_A: R65.2, U11.13 (THER)
- new net THER_B: R66.2, U12.13 (THER)
- no-connect marks 9 -> 16
Other:
- moved on the sheet: C41, C42, C43, C44, C45, C46, D10, D8, D9, J4, J8, R40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
