File: hardware/mccan.kicad_pcb (KiCad board)
At the start: 8 copper layers, 200 x 140 mm, 238 parts, among them J1 PWR pigtail -> SS1.5 3w, J2 Prog/UART, J3 FL pigtail -> SS1.0 key A / b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, J4 FR pigtail -> SS1.0 key B / g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, J5 RL pigtail -> SS1.0 key C / b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, J6 RR pigtail -> SS1.0 key D / n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, J7 DENALI pigtail -> SS1.5 3w, J8 CAN pigtail -> SS1.0 2w, Q10 IPT008N06NM5LF, Q11 IPT008N06NM5LF, Q12 MMBT3904, Q2 MMBT3904, Q3 MMBT3904, Q4 NX5020UNBKS, Q5 NX5020UNBKS, Q6 NX5020UNBKS, Q7 NX5020UNBKS, Q8 NX5020UNBKS, Q9 NX5020UNBKS, SW1 BOOT, SW2 EN/RESET, U1 LM5164DDA, U10 LTC4380HMS-2, U2 LM5164DDA, U3 LM51571-Q1, U4 DML3017LDC, U5 ESP32-WROOM-32E-N8, U6 TJA1042T/3, U7 PCA9685PW/Q900, U8 ADG706, U9 BTS7008-2EPA

Commit message: hw(pcb): CAN as a buried stripline on In2.Cu
Between the In1.Cu and In3.Cu ground planes, so segregation from the feed and the
switch node is structural -- the pair is physically enclosed in copper -- rather than
a keep-away rule nothing enforces. There is a ground plane between the
pair and every aggressor on the board, which matters more than connector spacing: J8 is
third in the gland row and 36.55 mm from J1, and that order is fixed by the enclosure.

Four nets, not two -- the choke splits each side, and Net-(U6-CANH/L) is the half that
reaches the transceiver.

Fix round 1 found three faults in the previous attempt (never regenerated, so its
"verified" comments cited a run that had not happened): the long haul crossing its own
pair partner, the J8 breakout converging between J8's own pads, and the R26 stub detour
checked against tracks but not vias. Landing the long haul on L6 instead of D6 (same net,
so electrically identical) fixes the first two; the D6/R26/L6 stubs and the L6->U6 hop
were re-routed around the vias fix round 1 found. The long haul's mid-board corridor also
turned up a field of ground-drop vias too dense for a single bump to clear -- solved with
an offline Dijkstra search over gen_pcb.py's own clearance functions rather than manual
tuning, documented in scripts/layout_pcb.py and task-8-report.md.

CANH 199.586 mm, CANL 174.368 mm, delta 25.219 mm.

Co-Authored-By: Claude Sonnet 5 <noreply@anthropic.com>
Routing:
- net /CANH: track 0.00 -> 199.6 mm, vias 0 -> 3
- net /CANL: track 0.00 -> 174.4 mm, vias 0 -> 5
- net Net-(U6-CANL): track 0.00 -> 42.5 mm, vias 0 -> 2
- net Net-(U6-CANH): track 0.00 -> 33.4 mm, vias 0 -> 2
